File: Untitled/Aeolus.kicad_sch (KiCad schematic)
At the start: 11 parts, among them J1 IR Receiver, J2 OLED Display, Q1 PN2222, SW1 SW_Push, U1 ESP32 - C3

Commit message: Add KiCad hardware design, branding, and full README
- Add Aeolus schematic, 4-layer PCB, custom footprints (ESP32-C3
  SuperMini, OLED, silkscreen logo) and 3D models
- Fix IR LED 3D model references to a shipping KiCad model
- Add branding artwork (logo/silk SVG + PNG)
- Rewrite README: project overview, hardware, firmware, pin map,
  PCB notes, and design improvements over the v1 fans project
- Remove leftover Untitled.* project files and gitignore KiCad
  backups/caches
Parts:
- D1, D2: footprint (none) -> LED_SMD:LED_PLCC-2_3.4x3.0mm_KA
- J1: footprint (none) -> OptoDevice:Vishay_MINICAST-3Pin
- J2: footprint (none) -> Aeolus_footprints:OLED_SSD1306_I2C_0.96
- Q1: footprint (none) -> Package_TO_SOT_THT:TO-92
- R1, R3: footprint (none) -> Resistor_SMD:R_0805_2012Metric
- R2: footprint (none) -> Resistor_SMD:R_2512_6332Metric
- SW1: footprint (none) -> Button_Switch_THT:SW_PUSH_6mm
- TH1: footprint (none) -> Capacitor_THT:C_Disc_D3.0mm_W1.6mm_P2.50mm
- U1: footprint (none) -> Aeolus_footprints:ESP32-C3-SuperMini
Changed lines of the file:
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@@
 			)
 		)
-		(property "Footprint" ""
+		(property "Footprint" "Package_TO_SOT_THT:TO-92"
 			(at 50.8 81.28 0)
 			(effects
@@
 			)
 		)
-		(property "Footprint" ""
+		(property "Footprint" "OptoDevice:Vishay_MINICAST-3Pin"
 			(at 182.88 93.98 0)
 			(effects
@@
 			)
 		)
-		(property "Footprint" ""
+		(property "Footprint" "Capacitor_THT:C_Disc_D3.0mm_W1.6mm_P2.50mm"
 			(at 167.64 123.19 0)
 			(effects
@@
 			)
 		)
-		(property "Footprint" ""
+		(property "Footprint" "Aeolus_footprints:ESP32-C3-SuperMini"
 			(at 144.78 92.71 0)
 			(effects
@@
 			)
 		)
-		(property "Footprint" ""
+		(property "Footprint" "Resistor_SMD:R_0805_2012Metric"
 			(at 129.54 83.058 90)
 			(effects
@@
 			)
 		)
-		(property "Footprint" ""
+		(property "Footprint" "Button_Switch_THT:SW_PUSH_6mm"
 			(at 106.68 107.95 0)
 			(effects
@@
 			)
 		)
-		(property "Footprint" ""
+		(property "Footprint" "LED_SMD:LED_PLCC-2_3.4x3.0mm_KA"
 			(at 105.41 95.25 0)
 			(effects
@@
 			)
 		)
-		(property "Footprint" ""
+		(property "Footprint" "LED_SMD:LED_PLCC-2_3.4x3.0mm_KA"
 			(at 113.03 95.25 0)
 			(effects
@@
 			)
 		)
-		(property "Footprint" ""
+		(property "Footprint" "Aeolus_footprints:OLED_SSD1306_I2C_0.96"
 			(at 114.3 123.19 0)
 			(effects
@@
 			)
 		)
-		(property "Footprint" ""
+		(property "Footprint" "Resistor_SMD:R_2512_6332Metric"
 			(at 120.65 97.028 90)
 			(effects
@@
 			)
 		)
-		(property "Footprint" ""
+		(property "Footprint" "Resistor_SMD:R_0805_2012Metric"
 			(at 165.862 114.3 90)
 			(effects
